Commit message: added arms

File: src/boxxo_core/urdf/boxxo.urdf.xacro (robot description, xacro)
@@ -2,4 +2,5 @@
 <robot name="boxxo" xmlns:xacro="http://www.ros.org/wiki/xacro">
 	<xacro:include filename="$(find boxxo_core)/urdf/wheel.urdf.xacro"/>
+	<xacro:include filename="$(find boxxo_core)/urdf/boxxo_arm.urdf.xacro"/>
     <!-- Chassis Properties -->
 	<xacro:property name="chassis_length" value="1.6256"/>
@@ -14,4 +15,8 @@
 	<xacro:property name="wheel_y_spacing" value="${chassis_width/2}"/>
 	<xacro:property name="wheel_z_spacing" value="${chassis_height/4}"/>
+	<!-- Arm Location -->
+	<xacro:property name="boxxo_arm_x" value=".2064"/>
+	<xacro:property name="boxxo_arm_y" value=".3"/>
+	<xacro:property name="boxxo_arm_z" value=".4"/>
 	<link name="base_link"/>
 	<!-- The chassis of the rover -->
@@ -55,3 +60,9 @@
 		<inertia ixx="0.08" ixy="0.0" ixz="0.0" iyy="0.14" iyz="0.0" izz="0.08"/>
 	</xacro:wheel>
+	<xacro:boxxo_arm endeffector="" prefix="left" parent="chassie">
+		<origin xyz="${boxxo_arm_x} ${boxxo_arm_y} ${boxxo_arm_z}" rpy="0 0 0"/>
+	</xacro:boxxo_arm>
+	<xacro:boxxo_arm endeffector="" prefix="right" parent="chassie">
+		<origin xyz="${boxxo_arm_x} -${boxxo_arm_y} ${boxxo_arm_z}" rpy="0 0 0"/>
+	</xacro:boxxo_arm>
 </robot>

Commit message: added cmaera

File: src/boxxo_core/urdf/boxxo.urdf.xacro (robot description, xacro)
@@ -3,9 +3,10 @@
 	<xacro:include filename="$(find boxxo_core)/urdf/wheel.urdf.xacro"/>
 	<xacro:include filename="$(find boxxo_core)/urdf/boxxo_arm.urdf.xacro"/>
+	<xacro:include filename="$(find boxxo_core)/urdf/camera.urdf.xacro"/>
     <!-- Chassis Properties -->
 	<xacro:property name="chassis_length" value="1.6256"/>
 	<xacro:property name="chassis_width" value="1.2446"/>
 	<xacro:property name="chassis_height" value="0.25"/>
-	<xacro:property name="chassis_mass" value="0"/>
+	<xacro:property name="chassis_mass" value="200"/>
 	<!-- Wheel Properties -->
 	<xacro:property name="wheel_depth" value="0.1286"/>
@@ -60,9 +61,12 @@
 		<inertia ixx="0.08" ixy="0.0" ixz="0.0" iyy="0.14" iyz="0.0" izz="0.08"/>
 	</xacro:wheel>
-	<xacro:boxxo_arm endeffector="" prefix="left" parent="chassie">
+	<xacro:boxxo_arm endeffector="camera" prefix="left" parent="chassie">
 		<origin xyz="${boxxo_arm_x} ${boxxo_arm_y} ${boxxo_arm_z}" rpy="0 0 0"/>
 	</xacro:boxxo_arm>
-	<xacro:boxxo_arm endeffector="" prefix="right" parent="chassie">
+	<xacro:boxxo_arm endeffector="camera" prefix="right" parent="chassie">
 		<origin xyz="${boxxo_arm_x} -${boxxo_arm_y} ${boxxo_arm_z}" rpy="0 0 0"/>
 	</xacro:boxxo_arm>
+	<xacro:boxxo_camera prefix="body" parent="chassie">
+		<origin xyz="${chassis_length/2-0.04} 0.25 ${chassis_height+0.02}" rpy="0 0 0"/>
+	</xacro:boxxo_camera>
 </robot>

File: src/boxxo_core/urdf/boxxo_arm.urdf.xacro (robot description, xacro)
@@ -1,5 +1,5 @@
 <?xml version="1.0"?>
 <robot name="boxxo_arm" xmlns:xacro="https://wiki.ros.org/xacro">
-	<!-- <xacro:include filename=""/> -->
+	<xacro:include filename="$(find boxxo_core)/urdf/camera.urdf.xacro"/>
 	<xacro:macro name="boxxo_arm" params="endeffector prefix parent *origin">
 		<xacro:property name="motor_height" value=".15"/>
@@ -191,4 +191,10 @@
 			<limit lower="-3.14" upper="3.14" velocity=".25" effort="300"/>
 		</joint>
+		<!-- ENDEFFECTOR IF STATEMENT -->
+		<xacro:if value="${endeffector == 'camera'}">
+			<xacro:boxxo_camera prefix="${prefix}" parent="${prefix}_j5_link">
+				<origin xyz="0 0 ${ee_length}" rpy="0 -1.57079632679 0"/>
+			</xacro:boxxo_camera>
+		</xacro:if>
 		<!-- TRANSMISSIONS -->
 		<transmission name="${prefix}_j1">
